File: kicad/mk2/srvant-mk2/interconnection.kicad_sch (KiCad schematic)
At the start: 0 parts

Commit message: more progress
Other:
- note added: "EEPROM_nWP: pull this pin low to disable changing EEPROM BT_nDisable: When driven, or tied low, it prevents the Bluetooth module from powering u WL_nDisable: When driven or tied low it prevents the wireless network module from powering up."
Changed lines of the file:
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@@
+    (stroke (width 0) (type default))
+  )
+  (wire (pts (xy 118.11 146.05) (xy 135.89 146.05))
     (stroke (width 0) (type default))
   )
@@
     (stroke (width 0) (type default))
   )
+  (wire (pts (xy 133.35 99.06) (xy 147.32 99.06))
+    (stroke (width 0) (type default))
+  )
+  (wire (pts (xy 133.35 93.98) (xy 147.32 93.98))
+    (stroke (width 0) (type default))
+  )
+  (wire (pts (xy 118.11 148.59) (xy 135.89 148.59))
+    (stroke (width 0) (type default))
+  )
+  (wire (pts (xy 133.35 96.52) (xy 147.32 96.52))
+    (stroke (width 0) (type default))
+  )
+  (wire (pts (xy 118.11 143.51) (xy 135.89 143.51))
+    (stroke (width 0) (type default))
+  )
+  (text "EEPROM_nWP: pull this pin low to disable changing EEPROM\nBT_nDisable: When driven, or tied low, it prevents the Bluetooth module from powering u\nWL_nDisable: When driven or tied low it prevents the wireless network module from powering up."
+    (at 96.52 139.7 0)
+    (effects (font (size 1.27 1.27)) (justify left bottom))
+  )
+  (hierarchical_label "BMC_HOST_WL_nDis" (shape input) (at 118.11 146.05 180) (fields_autoplaced)
+    (effects (font (size 1.27 1.27)) (justify right))
+  )
+  (hierarchical_label "BMC_HOST_POST_COMPLETE" (shape input) (at 118.11 166.37 180) (fields_autoplaced)
+    (effects (font (size 1.27 1.27)) (justify right))
+  )
   (hierarchical_label "BMC_UART0_TX" (shape input) (at 133.35 73.66 180) (fields_autoplaced)
+    (effects (font (size 1.27 1.27)) (justify right))
+  )
+  (hierarchical_label "BMC_HOST_USB_DEMUX_CONTROL" (shape input) (at 133.35 99.06 180) (fields_autoplaced)
     (effects (font (size 1.27 1.27)) (justify right))
   )
@@
     (effects (font (size 1.27 1.27)) (justify right))
   )
+  (hierarchical_label "HOST_WL_nDis" (shape output) (at 135.89 146.05 0) (fields_autoplaced)
+    (effects (font (size 1.27 1.27)) (justify left))
+  )
+  (hierarchical_label "BMC_HOST_POWER_OUT" (shape input) (at 118.11 163.83 180) (fields_autoplaced)
+    (effects (font (size 1.27 1.27)) (justify right))
+  )
+  (hierarchical_label "BMC_USB_HOST_N" (shape input) (at 133.35 96.52 180) (fields_autoplaced)
+    (effects (font (size 1.27 1.27)) (justify right))
+  )
   (hierarchical_label "HOST_UART_RX" (shape input) (at 144.78 73.66 0) (fields_autoplaced)
     (effects (font (size 1.27 1.27)) (justify left))
+  )
+  (hierarchical_label "HOST_BT_nDis" (shape output) (at 135.89 148.59 0) (fields_autoplaced)
+    (effects (font (size 1.27 1.27)) (justify left))
+  )
+  (hierarchical_label "BMC_HOST_RESET_OUT" (shape input) (at 118.11 161.29 180) (fields_autoplaced)
+    (effects (font (size 1.27 1.27)) (justify right))
+  )
+  (hierarchical_label "BMC_HOST_BT_nDis" (shape input) (at 118.11 148.59 180) (fields_autoplaced)
+    (effects (font (size 1.27 1.27)) (justify right))
+  )
+  (hierarchical_label "HOST_USB_P" (shape input) (at 147.32 93.98 0) (fields_autoplaced)
+    (effects (font (size 1.27 1.27)) (justify left))
+  )
+  (hierarchical_label "HOST_EEPROM_nWP" (shape output) (at 135.89 143.51 0) (fields_autoplaced)
+    (effects (font (size 1.27 1.27)) (justify left))
+  )
+  (hierarchical_label "BMC_USB_HOST_P" (shape input) (at 133.35 93.98 180) (fields_autoplaced)
+    (effects (font (size 1.27 1.27)) (justify right))
   )
   (hierarchical_label "HOST_UART_TX" (shape input) (at 144.78 71.12 0) (fields_autoplaced)
@@
     (effects (font (size 1.27 1.27)) (justify left))
   )
+  (hierarchical_label "BMC_HOST_EEPROM_nWP" (shape input) (at 118.11 143.51 180) (fields_autoplaced)
+    (effects (font (size 1.27 1.27)) (justify right))
+  )
+  (hierarchical_label "USB_DEMUX_SELECT" (shape input) (at 147.32 99.06 0) (fields_autoplaced)
+    (effects (font (size 1.27 1.27)) (justify left))
+  )
+  (hierarchical_label "HOST_USB_N" (shape input) (at 147.32 96.52 0) (fields_autoplaced)
+    (effects (font (size 1.27 1.27)) (justify left))
+  )
+  (hierarchical_label "BMC_HOST_nRPIBOOT" (shape input) (at 118.11 158.75 180) (fields_autoplaced)
+    (effects (font (size 1.27 1.27)) (justify right))
+  )
   (hierarchical_label "HOST_SCL_2" (shape input) (at 144.78 82.55 0) (fields_autoplaced)

Commit message: save state
Other:
- note removed: "EEPROM_nWP: pull this pin low to disable changing EEPROM BT_nDisable: When driven, or tied low, it prevents the Bluetooth module from powering u WL_nDisable: When driven or tied low it prevents the wireless network module from powering up."
Changed lines of the file:
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@@
     (rev "0.1")
-  )
-  (wire (pts (xy 133.35 82.55) (xy 144.78 82.55))
-    (stroke (width 0) (type default))
-  )
-  (wire (pts (xy 133.35 71.12) (xy 144.78 71.12))
-    (stroke (width 0) (type default))
-  )
-  (wire (pts (xy 118.11 146.05) (xy 135.89 146.05))
-    (stroke (width 0) (type default))
-  )
-  (wire (pts (xy 133.35 73.66) (xy 144.78 73.66))
-    (stroke (width 0) (type default))
-  )
-  (wire (pts (xy 133.35 85.09) (xy 144.78 85.09))
-    (stroke (width 0) (type default))
-  )
-  (wire (pts (xy 133.35 99.06) (xy 147.32 99.06))
-    (stroke (width 0) (type default))
-  )
-  (wire (pts (xy 133.35 93.98) (xy 147.32 93.98))
-    (stroke (width 0) (type default))
-  )
-  (wire (pts (xy 118.11 148.59) (xy 135.89 148.59))
-    (stroke (width 0) (type default))
-  )
-  (wire (pts (xy 133.35 96.52) (xy 147.32 96.52))
-    (stroke (width 0) (type default))
-  )
-  (wire (pts (xy 118.11 143.51) (xy 135.89 143.51))
-    (stroke (width 0) (type default))
-  )
-  (text "EEPROM_nWP: pull this pin low to disable changing EEPROM\nBT_nDisable: When driven, or tied low, it prevents the Bluetooth module from powering u\nWL_nDisable: When driven or tied low it prevents the wireless network module from powering up."
-    (at 96.52 139.7 0)
-    (effects (font (size 1.27 1.27)) (justify left bottom))
-  )
-  (hierarchical_label "BMC_HOST_WL_nDis" (shape input) (at 118.11 146.05 180) (fields_autoplaced)
-    (effects (font (size 1.27 1.27)) (justify right))
   )
   (hierarchical_label "BMC_HOST_POST_COMPLETE" (shape input) (at 118.11 166.37 180) (fields_autoplaced)
     (effects (font (size 1.27 1.27)) (justify right))
   )
-  (hierarchical_label "BMC_UART0_TX" (shape input) (at 133.35 73.66 180) (fields_autoplaced)
-    (effects (font (size 1.27 1.27)) (justify right))
-  )
-  (hierarchical_label "BMC_HOST_USB_DEMUX_CONTROL" (shape input) (at 133.35 99.06 180) (fields_autoplaced)
-    (effects (font (size 1.27 1.27)) (justify right))
-  )
-  (hierarchical_label "BMC_I2C_1_SDA" (shape output) (at 133.35 85.09 180) (fields_autoplaced)
-    (effects (font (size 1.27 1.27)) (justify right))
-  )
-  (hierarchical_label "BMC_I2C_1_SCK" (shape output) (at 133.35 82.55 180) (fields_autoplaced)
-    (effects (font (size 1.27 1.27)) (justify right))
-  )
-  (hierarchical_label "HOST_WL_nDis" (shape output) (at 135.89 146.05 0) (fields_autoplaced)
-    (effects (font (size 1.27 1.27)) (justify left))
-  )
   (hierarchical_label "BMC_HOST_POWER_OUT" (shape input) (at 118.11 163.83 180) (fields_autoplaced)
     (effects (font (size 1.27 1.27)) (justify right))
-  )
-  (hierarchical_label "BMC_USB_HOST_N" (shape input) (at 133.35 96.52 180) (fields_autoplaced)
-    (effects (font (size 1.27 1.27)) (justify right))
-  )
-  (hierarchical_label "HOST_UART_RX" (shape input) (at 144.78 73.66 0) (fields_autoplaced)
-    (effects (font (size 1.27 1.27)) (justify left))
-  )
-  (hierarchical_label "HOST_BT_nDis" (shape output) (at 135.89 148.59 0) (fields_autoplaced)
-    (effects (font (size 1.27 1.27)) (justify left))
   )
   (hierarchical_label "BMC_HOST_RESET_OUT" (shape input) (at 118.11 161.29 180) (fields_autoplaced)
     (effects (font (size 1.27 1.27)) (justify right))
   )
-  (hierarchical_label "BMC_HOST_BT_nDis" (shape input) (at 118.11 148.59 180) (fields_autoplaced)
-    (effects (font (size 1.27 1.27)) (justify right))
-  )
-  (hierarchical_label "HOST_USB_P" (shape input) (at 147.32 93.98 0) (fields_autoplaced)
-    (effects (font (size 1.27 1.27)) (justify left))
-  )
-  (hierarchical_label "HOST_EEPROM_nWP" (shape output) (at 135.89 143.51 0) (fields_autoplaced)
-    (effects (font (size 1.27 1.27)) (justify left))
-  )
-  (hierarchical_label "BMC_USB_HOST_P" (shape input) (at 133.35 93.98 180) (fields_autoplaced)
-    (effects (font (size 1.27 1.27)) (justify right))
-  )
-  (hierarchical_label "HOST_UART_TX" (shape input) (at 144.78 71.12 0) (fields_autoplaced)
-    (effects (font (size 1.27 1.27)) (justify left))
-  )
-  (hierarchical_label "HOST_SDA_2" (shape input) (at 144.78 85.09 0) (fields_autoplaced)
-    (effects (font (size 1.27 1.27)) (justify left))
-  )
-  (hierarchical_label "BMC_HOST_EEPROM_nWP" (shape input) (at 118.11 143.51 180) (fields_autoplaced)
-    (effects (font (size 1.27 1.27)) (justify right))
-  )
-  (hierarchical_label "USB_DEMUX_SELECT" (shape input) (at 147.32 99.06 0) (fields_autoplaced)
-    (effects (font (size 1.27 1.27)) (justify left))
-  )
-  (hierarchical_label "HOST_USB_N" (shape input) (at 147.32 96.52 0) (fields_autoplaced)
-    (effects (font (size 1.27 1.27)) (justify left))
-  )
   (hierarchical_label "BMC_HOST_nRPIBOOT" (shape input) (at 118.11 158.75 180) (fields_autoplaced)
     (effects (font (size 1.27 1.27)) (justify right))
   )
-  (hierarchical_label "HOST_SCL_2" (shape input) (at 144.78 82.55 0) (fields_autoplaced)
-    (effects (font (size 1.27 1.27)) (justify left))
-  )
-  (hierarchical_label "BMC_UART0_RX" (shape input) (at 133.35 71.12 180) (fields_autoplaced)
-    (effects (font (size 1.27 1.27)) (justify right))
-  )
