File: kicad/mk2/srvant-mk2/cm4_gpio.kicad_sch (KiCad schematic)
At the start: 13 parts, among them J4 ARJM11, U7 74LVC1G07SE-7, U8 TPD4EUSB30, U9 TPD4EUSB30

Commit message: more progress
Parts:
- added C76: 100n, Capacitor_SMD:C_0402_1005Metric, symbol Device:C
- added FB6: 220R, Resistor_SMD:R_0402_1005Metric, symbol Device:FerriteBead_Small
Connections:
- net GND: now also C76.2, FB6.2; no longer J4.SH
- net at C35.1, J4.5 (CT), J4.6 (CT): now also C76.1
- new net: FB6.1, J4.SH
Changed lines of the file:
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@@
   (junction (at 116.84 85.09) (diameter 1.016) (color 0 0 0 0)
   )
+  (junction (at 344.17 50.8) (diameter 0) (color 0 0 0 0)
+  )
   (junction (at 116.84 113.03) (diameter 1.016) (color 0 0 0 0)
   )
@@
   )
   (junction (at 53.34 46.99) (diameter 1.016) (color 0 0 0 0)
+  )
+  (junction (at 344.17 59.69) (diameter 0) (color 0 0 0 0)
   )
   (junction (at 115.57 128.27) (diameter 1.016) (color 0 0 0 0)
@@
     (stroke (width 0) (type solid))
   )
+  (wire (pts (xy 337.82 50.8) (xy 337.82 52.07))
+    (stroke (width 0) (type default))
+  )
   (wire (pts (xy 40.64 90.17) (xy 54.61 90.17))
     (stroke (width 0) (type solid))
@@
     (stroke (width 0) (type solid))
   )
+  (wire (pts (xy 378.46 85.09) (xy 378.46 87.63))
+    (stroke (width 0) (type default))
+  )
   (wire (pts (xy 51.2572 146.05) (xy 54.61 146.05))
     (stroke (width 0) (type solid))
@@
     (stroke (width 0) (type solid))
   )
+  (wire (pts (xy 378.46 92.71) (xy 378.46 93.98))
+    (stroke (width 0) (type default))
+  )
   (wire (pts (xy 116.84 144.78) (xy 120.2182 144.78))
     (stroke (width 0) (type solid))
@@
     (stroke (width 0) (type solid))
   )
+  (wire (pts (xy 344.17 60.96) (xy 344.17 59.69))
+    (stroke (width 0) (type default))
+  )
   (wire (pts (xy 115.57 31.75) (xy 116.84 31.75))
     (stroke (width 0) (type solid))
@@
     (stroke (width 0) (type solid))
   )
+  (wire (pts (xy 337.82 59.69) (xy 344.17 59.69))
+    (stroke (width 0) (type default))
+  )
   (wire (pts (xy 115.57 72.39) (xy 116.84 72.39))
     (stroke (width 0) (type solid))
@@
     (stroke (width 0) (type solid))
   )
-  (wire (pts (xy 378.46 85.09) (xy 378.46 90.17))
-    (stroke (width 0) (type solid))
-  )
   (polyline (pts (xy 279.4 21.59) (xy 394.97 21.59))
     (stroke (width 0) (type solid))
@@
   (wire (pts (xy 116.84 105.41) (xy 116.84 113.03))
     (stroke (width 0) (type solid))
+  )
+  (wire (pts (xy 344.17 50.8) (xy 337.82 50.8))
+    (stroke (width 0) (type default))
   )
   (wire (pts (xy 115.57 128.27) (xy 115.57 130.81))
@@
     )
   )
-  (symbol (lib_id "power:GND") (at 378.46 90.17 0) (unit 1)
+  (symbol (lib_id "power:GND") (at 378.46 93.98 0) (unit 1)
     (in_bom yes) (on_board yes) (dnp no)
-    (property "Reference" "#PWR032" (at 378.46 96.52 0)
-      (effects (font (size 1.27 1.27)) hide)
-    )
-    (property "Value" "GND" (at 378.587 94.5642 0)
+    (property "Reference" "#PWR032" (at 378.46 100.33 0)
+      (effects (font (size 1.27 1.27)) hide)
+    )
+    (property "Value" "GND" (at 378.587 98.3742 0)
       (effects (font (size 1.27 1.27)))
     )
-    (property "Footprint" "" (at 378.46 90.17 0)
-      (effects (font (size 1.27 1.27)) hide)
-    )
-    (property "Datasheet" "" (at 378.46 90.17 0)
+    (property "Footprint" "" (at 378.46 93.98 0)
+      (effects (font (size 1.27 1.27)) hide)
+    )
+    (property "Datasheet" "" (at 378.46 93.98 0)
       (effects (font (size 1.27 1.27)) hide)
     )
@@
     )
   )
+  (symbol (lib_id "Device:FerriteBead_Small") (at 378.46 90.17 0) (unit 1)
+    (in_bom yes) (on_board yes) (dnp no)
+    (property "Reference" "FB6" (at 375.92 90.17 90)
+      (effects (font (size 1.27 1.27)))
+    )
+    (property "Value" "220R" (at 382.27 90.17 90)
+      (effects (font (size 1.27 1.27)))
+    )
+    (property "Footprint" "Resistor_SMD:R_0402_1005Metric" (at 376.682 90.17 90)
+      (effects (font (size 1.27 1.27)) hide)
+    )
+    (property "Datasheet" "https://www.mouser.co.uk/datasheet/2/281/1/Murata_4_42023_QNFA9103SH-3135182.pdf" (at 378.46 90.17 0)
+      (effects (font (size 1.27 1.27)) hide)
+    )
+    (property "manf#" "BLM15PX221SH1D " (at 378.46 90.17 0)
+      (effects (font (size 1.27 1.27)) hide)
+    )
+    (property "digikey#" "" (at 378.46 90.17 0)
+      (effects (font (size 1.27 1.27)) hide)
+    )
+    (property "mouser#" " 81-BLM15PX221SH1D " (at 378.46 90.17 0)
+      (effects (font (size 1.27 1.27)) hide)
+    )
+    (property "farnell#" "" (at 378.46 90.17 0)
+      (effects (font (size 1.27 1.27)) hide)
+    )
+    (property "rs#" "" (at 378.46 90.17 0)
+      (effects (font (size 1.27 1.27)) hide)
+    )
+    (property "Part Description" "" (at 378.46 90.17 0)
+      (effects (font (size 1.27 1.27)) hide)
+    )
+    (pin "1")
+    (pin "2")
+    (instances
+      (project "srvant-mk2"
+        (path "/1859a578-b791-4142-bdf4-fda494df1146/a3ddce6d-c94c-48a5-9fee-a70fbee730bf"
+          (reference "FB6") (unit 1)
+        )
+        (path "/1859a578-b791-4142-bdf4-fda494df1146/75d0860a-7ab5-4d7d-b96d-9266ebc33987/5816e81d-55cb-47d6-914e-ed3118b5e71f"
+          (reference "FB7") (unit 1)
+        )
+      )
+    )
+  )
   (symbol (lib_id "power:GND") (at 309.88 50.8 0) (unit 1)
     (in_bom yes) (on_board yes) (dnp no)
@@
     )
   )
-  (symbol (lib_id "power:GND") (at 344.17 59.69 0) (unit 1)
+  (symbol (lib_id "power:GND") (at 344.17 60.96 0) (unit 1)
     (in_bom yes) (on_board yes) (dnp no)
-    (property "Reference" "#PWR031" (at 344.17 66.04 0)
-      (effects (font (size 1.27 1.27)) hide)
-    )
-    (property "Value" "GND" (at 344.297 64.0842 0)
+    (property "Reference" "#PWR031" (at 344.17 67.31 0)
+      (effects (font (size 1.27 1.27)) hide)
+    )
+    (property "Value" "GND" (at 344.297 65.3542 0)
       (effects (font (size 1.27 1.27)))
     )
-    (property "Footprint" "" (at 344.17 59.69 0)
-      (effects (font (size 1.27 1.27)) hide)
-    )
-    (property "Datasheet" "" (at 344.17 59.69 0)
+    (property "Footprint" "" (at 344.17 60.96 0)
+      (effects (font (size 1.27 1.27)) hide)
+    )
+    (property "Datasheet" "" (at 344.17 60.96 0)
       (effects (font (size 1.27 1.27)) hide)
     )
@@
         )
       )
+    )
+  )
+  (symbol (lib_id "Device:C") (at 337.82 55.88 0) (unit 1)
+    (in_bom yes) (on_board yes) (dnp no)
+    (property "Reference" "C76" (at 340.741 54.7116 0)
+      (effects (font (size 1.27 1.27)) (justify left))
+    )
+    (property "Value" "100n" (at 340.741 57.023 0)
+      (effects (font (size 1.27 1.27)) (justify left))
+    )
+    (property "Footprint" "Capacitor_SMD:C_0402_1005Metric" (at 338.7852 59.69 0)
+      (effects (font (size 1.27 1.27)) hide)
+    )
+    (property "Datasheet" "https://search.murata.co.jp/Ceramy/image/img/A01X/G101/ENG/GRM155R71C104KA88-01.pdf" (at 337.82 55.88 0)
+      (effects (font (size 1.27 1.27)) hide)
+    )
+    (property "Field4" "Farnell" (at 337.82 55.88 0)
+      (effects (font (size 1.27 1.27)) hide)
+    )
+    (property "Field5" "2611911" (at 337.82 55.88 0)
+      (effects (font (size 1.27 1.27)) hide)
+    )
+    (property "Field6" "RM EMK105 B7104KV-F" (at 337.82 55.88 0)
+      (effects (font (size 1.27 1.27)) hide)
+    )
+    (property "Field7" "TAIYO YUDEN EUROPE GMBH" (at 337.82 55.88 0)
+      (effects (font (size 1.27 1.27)) hide)
+    )
+    (property "Part Description" "	0.1uF 10% 16V Ceramic Capacitor X7R 0402 (1005 Metric)" (at 337.82 55.88 0)
+      (effects (font (size 1.27 1.27)) hide)
+    )
+    (property "Field8" "110091611" (at 337.82 55.88 0)
+      (effects (font (size 1.27 1.27)) hide)
+    )
+    (pin "1")
+    (pin "2")
+    (instances
+      (project "srvant-mk2"
+        (path "/1859a578-b791-4142-bdf4-fda494df1146/75d0860a-7ab5-4d7d-b96d-9266ebc33987/5816e81d-55cb-47d6-914e-ed3118b5e71f"
+          (reference "C76") (unit 1)
+        )
+      )
+      (project "srvant"
+        (path "/556fa623-1b37-4e79-bae4-da8a8b5c51e2/e09acda0-94a3-4a08-aefe-d9a65d235818/4ef40d64-4bce-4f26-8bb0-6b5010a92d45"
+          (reference "C119") (unit 1)
+        )
+      )

Commit message: add rp-t113-s3 datasheets (cn), make CI happier
Parts:
- C35, C76: Part Description 0.1uF 10% 16V Ceramic Capacitor X7R 0402 (1005 Metric) -> 0.1uF 10% 16V Ceramic Capacitor X7R 0402 (1005 Metric)
- D2: Field4 Digikey -> Digikey; Part Description Green 572nm LED Indication - Discrete 2.2V 2-SMD, No Lead -> Green 572nm LED Indication - Discrete 2.2V 2-SMD, No Lead
- D3: Field4 Digikey -> Digikey; Field5 LTST-S270KRKT -> LTST-S270KRKT; Part Description Red 620nm LED Indication - Discrete 2.2V 2-SMD, No Lead -> Red 620nm LED Indication - Discrete 2.2V 2-SMD, No Lead
- FB6: manf# BLM15PX221SH1D -> BLM15PX221SH1D; mouser# 81-BLM15PX221SH1D -> 81-BLM15PX221SH1D
- Module1: Part Description 100 Position Connector Receptacle, Center Strip Contacts Surface Mount Gold -> 100 Position Connector Receptacle, Center Strip Contacts Surface Mount Gold
- R13, R14: Field6 RK73G1ETQTP4700D -> RK73G1ETQTP4700D
Changed lines of the file:
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@@
       (effects (font (size 1.27 1.27)) hide)
     )
-    (property "Field6" "RK73G1ETQTP4700D         " (at 346.71 77.47 0)
+    (property "Field6" "RK73G1ETQTP4700D" (at 346.71 77.47 0)
       (effects (font (size 1.27 1.27)) hide)
     )
@@
       (effects (font (size 1.27 1.27)) hide)
     )
-    (property "Field4" "Digikey " (at 342.9 213.36 0)
-      (effects (font (size 1.27 1.27)) hide)
-    )
-    (property "Field5" "	LTST-S270KRKT" (at 342.9 213.36 0)
+    (property "Field4" "Digikey" (at 342.9 213.36 0)
+      (effects (font (size 1.27 1.27)) hide)
+    )
+    (property "Field5" "LTST-S270KRKT" (at 342.9 213.36 0)
       (effects (font (size 1.27 1.27)) hide)
     )
@@
       (effects (font (size 1.27 1.27)) hide)
     )
-    (property "Part Description" "	Red 620nm LED Indication - Discrete 2.2V 2-SMD, No Lead" (at 342.9 213.36 0)
+    (property "Part Description" "Red 620nm LED Indication - Discrete 2.2V 2-SMD, No Lead" (at 342.9 213.36 0)
       (effects (font (size 1.27 1.27)) hide)
     )
@@
       (effects (font (size 1.27 1.27)) hide)
     )
-    (property "Field6" "RK73G1ETQTP4700D         " (at 346.71 82.55 0)
+    (property "Field6" "RK73G1ETQTP4700D" (at 346.71 82.55 0)
       (effects (font (size 1.27 1.27)) hide)
     )
@@
       (effects (font (size 1.27 1.27)) hide)
     )
-    (property "Field4" "Digikey " (at 132.334 38.1 0)
+    (property "Field4" "Digikey" (at 132.334 38.1 0)
       (effects (font (size 1.27 1.27)) hide)
     )
@@
       (effects (font (size 1.27 1.27)) hide)
     )
-    (property "Part Description" "	Green 572nm LED Indication - Discrete 2.2V 2-SMD, No Lead" (at 132.334 38.1 0)
+    (property "Part Description" "Green 572nm LED Indication - Discrete 2.2V 2-SMD, No Lead" (at 132.334 38.1 0)
       (effects (font (size 1.27 1.27)) hide)
     )
@@
       (effects (font (size 1.27 1.27)) hide)
     )
-    (property "Part Description" "	0.1uF 10% 16V Ceramic Capacitor X7R 0402 (1005 Metric)" (at 344.17 55.88 0)
+    (property "Part Description" "0.1uF 10% 16V Ceramic Capacitor X7R 0402 (1005 Metric)" (at 344.17 55.88 0)
       (effects (font (size 1.27 1.27)) hide)
     )
@@
       (effects (font (size 1.27 1.27)) hide)
     )
-    (property "manf#" "BLM15PX221SH1D " (at 378.46 90.17 0)
+    (property "manf#" "BLM15PX221SH1D" (at 378.46 90.17 0)
       (effects (font (size 1.27 1.27)) hide)
     )
@@
       (effects (font (size 1.27 1.27)) hide)
     )
-    (property "mouser#" " 81-BLM15PX221SH1D " (at 378.46 90.17 0)
+    (property "mouser#" "81-BLM15PX221SH1D" (at 378.46 90.17 0)
       (effects (font (size 1.27 1.27)) hide)
     )
@@
       (effects (font (size 1.27 1.27)) hide)
     )
-    (property "Part Description" "	100 Position Connector Receptacle, Center Strip Contacts Surface Mount Gold" (at 87.63 87.63 0)
+    (property "Part Description" "100 Position Connector Receptacle, Center Strip Contacts Surface Mount Gold" (at 87.63 87.63 0)
       (effects (font (size 1.27 1.27)) hide)
     )
@@
       (effects (font (size 1.27 1.27)) hide)
     )
-    (property "Part Description" "	0.1uF 10% 16V Ceramic Capacitor X7R 0402 (1005 Metric)" (at 337.82 55.88 0)
-      (effects (font (size 1.27 1.27)) hide)
-    )
+    (property "Part Description" "0.1uF 10% 16V Ceramic Capacitor X7R 0402 (1005 Metric)" (at 337.82 55.88 0)
+      (effects (font (size 1.27 1.27)) hide)
+    )
