File: kicad/mk2/srvant-mk2/cm4_high_speed.kicad_sch (KiCad schematic)
At the start: 40 parts, among them J2 Bus_M.2_Socket_M, J3 690-019-298-412, U10 RT9742SNGV, U3 TLV62585DRLR, U4 BD2221G-LBTR, U5 PCF85063AT/AAZ, U6 74LVC1G07SE-7, Y1 X32K768S301

Commit message: more progress
Parts:
- removed C30, C31: 100n, Capacitor_SMD:C_0402_1005Metric, symbol Device:C
- removed R8: 100K/1%, Resistor_SMD:R_0402_1005Metric, symbol Device:R
- removed U4: BD2221G-LBTR, srvant:BD2221G-LBTR, symbol BD2221G-LBTR:BD2221G-LBTR
- J3: value 690-019-298-412 -> HDMI connector; footprint srvant:10029449-001RLF -> footprints:HDMI-10029449-001RLF; Field4 Farnell -> (none); Field5 2614936 -> (none); Field6 690-019-298-412 -> (none); Field7 EDAC -> (none); Field8 UCON00802 -> (none); farnell# (none) -> 2614936; manf# (none) -> 10029449-001RLF; rs# (none) -> 771-0094
- U3: footprint srvant:TLV62585DRLR -> TLV62585DRLR:DRL0006A; manf# (none) -> TLV62585DRLR; mouser# (none) -> 595-TLV62585DRLR
Other:
- note removed: "original CM4 board uses RT9742. Use it?"
- moved on the sheet: C36, C37, U10

Commit message: add rp-t113-s3 datasheets (cn), make CI happier
Parts:
- C19, C20: Field6 GRM21BC8YA106KE11L -> GRM21BC8YA106KE11L; Part Description 10uF 10% or 20% 35V Ceramic Capacitor X6S 0805 (2012 Metric) -> 10uF 10% or 20% 35V Ceramic Capacitor X6S 0805 (2012 Metric)
- C21, C22, C24, C25, C26, C28: Part Description 10uF 10% 10V Ceramic Capacitor X7R 0805 (2012 Metric) -> 10uF 10% 10V Ceramic Capacitor X7R 0805 (2012 Metric)
- C23, C27, C29, C32, C33, C34, C36, C37: Part Description 0.1uF 10% 16V Ceramic Capacitor X7R 0402 (1005 Metric) -> 0.1uF 10% 16V Ceramic Capacitor X7R 0402 (1005 Metric)
- Module1: Part Description 100 Position Connector Receptacle, Center Strip Contacts Surface Mount Gold -> 100 Position Connector Receptacle, Center Strip Contacts Surface Mount Gold
- R7: Field6 RK73G1ETQTP4702D -> RK73G1ETQTP4702D
- U3: manf# TLV62585DRLR -> TLV62585DRLR; mouser# 595-TLV62585DRLR -> 595-TLV62585DRLR
Changed lines of the file:
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@@
       (effects (font (size 1.27 1.27)) hide)
     )
-    (property "Part Description" "	0.1uF 10% 16V Ceramic Capacitor X7R 0402 (1005 Metric)" (at 330.2 -78.74 0)
+    (property "Part Description" "0.1uF 10% 16V Ceramic Capacitor X7R 0402 (1005 Metric)" (at 330.2 -78.74 0)
       (effects (font (size 1.27 1.27)) hide)
     )
@@
       (effects (font (size 1.27 1.27)) hide)
     )
-    (property "Part Description" "	0.1uF 10% 16V Ceramic Capacitor X7R 0402 (1005 Metric)" (at 364.49 -71.12 0)
+    (property "Part Description" "0.1uF 10% 16V Ceramic Capacitor X7R 0402 (1005 Metric)" (at 364.49 -71.12 0)
       (effects (font (size 1.27 1.27)) hide)
     )
@@
       (effects (font (size 1.524 1.524)) hide)
     )
-    (property "manf#" "TLV62585DRLR " (at 195.58 250.19 0)
+    (property "manf#" "TLV62585DRLR" (at 195.58 250.19 0)
       (effects (font (size 1.27 1.27)) hide)
     )
@@
       (effects (font (size 1.27 1.27)) hide)
     )
-    (property "mouser#" " 595-TLV62585DRLR " (at 195.58 250.19 0)
+    (property "mouser#" "595-TLV62585DRLR" (at 195.58 250.19 0)
       (effects (font (size 1.27 1.27)) hide)
     )
@@
       (effects (font (size 1.27 1.27)) hide)
     )
-    (property "Part Description" "	10uF 10% 10V Ceramic Capacitor X7R 0805 (2012 Metric)" (at 115.57 233.68 0)
+    (property "Part Description" "10uF 10% 10V Ceramic Capacitor X7R 0805 (2012 Metric)" (at 115.57 233.68 0)
       (effects (font (size 1.27 1.27)) hide)
     )
@@
       (effects (font (size 1.27 1.27)) hide)
     )
-    (property "Part Description" "	0.1uF 10% 16V Ceramic Capacitor X7R 0402 (1005 Metric)" (at 273.05 52.07 0)
+    (property "Part Description" "0.1uF 10% 16V Ceramic Capacitor X7R 0402 (1005 Metric)" (at 273.05 52.07 0)
       (effects (font (size 1.27 1.27)) hide)
     )
@@
       (effects (font (size 1.27 1.27)) hide)
     )
-    (property "Field6" "GRM21BC8YA106KE11L " (at 168.148 246.38 0)
+    (property "Field6" "GRM21BC8YA106KE11L" (at 168.148 246.38 0)
       (effects (font (size 1.27 1.27)) hide)
     )
@@
       (effects (font (size 1.27 1.27)) hide)
     )
-    (property "Part Description" "	10uF 10% or 20% 35V Ceramic Capacitor X6S 0805 (2012 Metric)" (at 168.148 246.38 0)
+    (property "Part Description" "10uF 10% or 20% 35V Ceramic Capacitor X6S 0805 (2012 Metric)" (at 168.148 246.38 0)
       (effects (font (size 1.27 1.27)) hide)
     )
@@
       (effects (font (size 1.27 1.27)) hide)
     )
-    (property "Part Description" "	100 Position Connector Receptacle, Center Strip Contacts Surface Mount Gold" (at -52.07 88.9 0)
+    (property "Part Description" "100 Position Connector Receptacle, Center Strip Contacts Surface Mount Gold" (at -52.07 88.9 0)
       (effects (font (size 1.27 1.27)) hide)
     )
@@
       (effects (font (size 1.27 1.27)) hide)
     )
-    (property "Part Description" "	0.1uF 10% 16V Ceramic Capacitor X7R 0402 (1005 Metric)" (at 339.598 -130.7846 0)
+    (property "Part Description" "0.1uF 10% 16V Ceramic Capacitor X7R 0402 (1005 Metric)" (at 339.598 -130.7846 0)
       (effects (font (size 1.27 1.27)) hide)
     )
@@
       (effects (font (size 1.27 1.27)) hide)
     )
-    (property "Part Description" "	0.1uF 10% 16V Ceramic Capacitor X7R 0402 (1005 Metric)" (at 124.46 260.35 0)
+    (property "Part Description" "0.1uF 10% 16V Ceramic Capacitor X7R 0402 (1005 Metric)" (at 124.46 260.35 0)
       (effects (font (size 1.27 1.27)) hide)
     )
@@
       (effects (font (size 1.27 1.27)) hide)
     )
-    (property "Part Description" "	0.1uF 10% 16V Ceramic Capacitor X7R 0402 (1005 Metric)" (at 306.07 52.07 0)
+    (property "Part Description" "0.1uF 10% 16V Ceramic Capacitor X7R 0402 (1005 Metric)" (at 306.07 52.07 0)
       (effects (font (size 1.27 1.27)) hide)
     )
@@
       (effects (font (size 1.27 1.27)) hide)
     )
-    (property "Part Description" "	10uF 10% 10V Ceramic Capacitor X7R 0805 (2012 Metric)" (at 265.684 237.998 0)
+    (property "Part Description" "10uF 10% 10V Ceramic Capacitor X7R 0805 (2012 Metric)" (at 265.684 237.998 0)
       (effects (font (size 1.27 1.27)) hide)
     )
@@
       (effects (font (size 1.27 1.27)) hide)
     )
-    (property "Part Description" "	10uF 10% 10V Ceramic Capacitor X7R 0805 (2012 Metric)" (at 255.524 237.998 0)
+    (property "Part Description" "10uF 10% 10V Ceramic Capacitor X7R 0805 (2012 Metric)" (at 255.524 237.998 0)
       (effects (font (size 1.27 1.27)) hide)
     )
@@
       (effects (font (size 1.27 1.27)) hide)
     )
-    (property "Part Description" "	10uF 10% 10V Ceramic Capacitor X7R 0805 (2012 Metric)" (at 116.078 205.74 0)
+    (property "Part Description" "10uF 10% 10V Ceramic Capacitor X7R 0805 (2012 Metric)" (at 116.078 205.74 0)
       (effects (font (size 1.27 1.27)) hide)
     )
@@
       (effects (font (size 1.27 1.27)) hide)
     )
-    (property "Part Description" "	0.1uF 10% 16V Ceramic Capacitor X7R 0402 (1005 Metric)" (at 124.46 233.68 0)
+    (property "Part Description" "0.1uF 10% 16V Ceramic Capacitor X7R 0402 (1005 Metric)" (at 124.46 233.68 0)
       (effects (font (size 1.27 1.27)) hide)
     )
@@
       (effects (font (size 1.27 1.27)) hide)
     )
-    (property "Part Description" "	10uF 10% 10V Ceramic Capacitor X7R 0805 (2012 Metric)" (at 115.57 260.35 0)
+    (property "Part Description" "10uF 10% 10V Ceramic Capacitor X7R 0805 (2012 Metric)" (at 115.57 260.35 0)
       (effects (font (size 1.27 1.27)) hide)
     )
@@
       (effects (font (size 1.27 1.27)) hide)
     )
-    (property "Field6" "RK73G1ETQTP4702D  " (at 234.188 249.936 0)
+    (property "Field6" "RK73G1ETQTP4702D" (at 234.188 249.936 0)
       (effects (font (size 1.27 1.27)) hide)
     )
@@
       (effects (font (size 1.27 1.27)) hide)
     )
-    (property "Part Description" "	10uF 10% 10V Ceramic Capacitor X7R 0805 (2012 Metric)" (at 245.364 237.998 0)
+    (property "Part Description" "10uF 10% 10V Ceramic Capacitor X7R 0805 (2012 Metric)" (at 245.364 237.998 0)
       (effects (font (size 1.27 1.27)) hide)
     )
@@
       (effects (font (size 1.27 1.27)) hide)
     )
-    (property "Field6" "GRM21BC8YA106KE11L " (at 160.274 246.38 0)
+    (property "Field6" "GRM21BC8YA106KE11L" (at 160.274 246.38 0)
       (effects (font (size 1.27 1.27)) hide)
     )
@@
       (effects (font (size 1.27 1.27)) hide)
     )
-    (property "Part Description" "	10uF 10% or 20% 35V Ceramic Capacitor X6S 0805 (2012 Metric)" (at 160.274 246.38 0)
+    (property "Part Description" "10uF 10% or 20% 35V Ceramic Capacitor X6S 0805 (2012 Metric)" (at 160.274 246.38 0)
       (effects (font (size 1.27 1.27)) hide)
     )
@@
       (effects (font (size 1.27 1.27)) hide)
     )
-    (property "Part Description" "	0.1uF 10% 16V Ceramic Capacitor X7R 0402 (1005 Metric)" (at 124.968 205.74 0)
-      (effects (font (size 1.27 1.27)) hide)
-    )
+    (property "Part Description" "0.1uF 10% 16V Ceramic Capacitor X7R 0402 (1005 Metric)" (at 124.968 205.74 0)
+      (effects (font (size 1.27 1.27)) hide)
+    )
