File: kicad/mk2/srvant-mk2/bmc_eth.kicad_sch (KiCad schematic)
At the start: 84 parts, among them J5 ARJM11, U10 TPD4EUSB30, U11 TPD4EUSB30, U12 KSZ9131RNXI-TR, U5 rp-t113-s3, Y2 25Mhz

Commit message: redesign for the next version
Parts:
- removed C58: 100n, Capacitor_SMD:C_0402_1005Metric, symbol Device:C
- removed C67, C68: 15p, Capacitor_SMD:C_0402_1005Metric, symbol Device:C
- removed FB3: 220R, Resistor_SMD:R_0402_1005Metric, symbol Device:FerriteBead_Small
- removed U5: rp-t113-s3, footprints:rp-t113-s3, symbol custom-libraries:t113-s3
- removed Y2: 25Mhz, PCM_Crystal_AKL:Crystal_SMD_FOX_FQ7050-4Pin_7.0x5.0mm, symbol Device:Crystal_GND24
- added C122, C123, C126: 100n, Capacitor_SMD:C_0402_1005Metric, symbol Device:C
- added C124: 10u, Capacitor_SMD:C_0402_1005Metric, symbol Device:C
- added C125: 1u, Capacitor_SMD:C_0402_1005Metric, symbol Device:C
- added MOSFET1: DMP3098LQ-7, DMP3098L:SOT-23_DMP3098LQ_DIO, symbol DMP3098L:DMP3098LQ-7
- added R79: 100K, Resistor_SMD:R_0402_1005Metric, symbol Device:R
Connections:
- net 1V2: now also C123.1, C124.1, C125.1, C126.1, MOSFET1.3 (D)
- net 3.3v_PHY: now also C55.1, C122.1, MOSFET1.2 (S), R79.1
- net EPHY_25M: now also U12.46 (XI)
- net GND: now also C122.2, C123.2, C124.2, C125.2, C126.2
- net LDO_OUT: now reaches U12.43 (LDO_O)
- net LDO_OUT: now also MOSFET1.1 (G), R79.2; no longer C55.1
- net +3.3v_BMC renamed +3v3_AUX
- net CLK125_OUT / LED_MODE renamed CLK125_OUT
- net RESET_OUT_N renamed MAC_RESET_OUT_N
Other:
- note added: "TODO: LDO output needs to be fixed! either add required components to use internal LDO or add external LDO"
- note removed: "Are these 22R resistors a must? Can I work around them by using required trace widths?"
- note removed: "RGMII_CLKIN: function unknown possibly needs to be connected to CLK125 of PHY"
- moved on the sheet: C33, C34, C35, C36, C38, C39, C41, C43, C45, C46, C47, C48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
