File: kicad/mk2/srvant-mk2/srvant-mk2.kicad_sch (KiCad schematic)
At the start: 4 parts

Commit message: redesign for the next version
Other:
- sheet BMC ethernet ports: added +3v3_AUX; removed +3.3v_BMC
- sheet bmc ports: added +3v3_AUX; removed +3.3v_BMC
- sheet cm4 ports: added +3v3_AUX; removed +3.3v_HOST_PCIe
- sheet power ports: added +3v3_AUX; removed +3.3v_BMC, +3.3v_HOST_PCIe
- note added: "Do i need 2 pins for the HOST_RUN_PG? should it be a single one?"
Changed lines of the file:
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@@
 		)
 		(stroke
-			(width 0)
-			(type default)
+			(width 1)
+			(type default)
+			(color 73 152 255 1)
 		)
 	)
@@
 	(wire
 		(pts
+			(xy 102.87 76.2) (xy 285.75 76.2)
+		)
+		(stroke
+			(width 1)
+			(type default)
+			(color 73 152 255 1)
+		)
+	)
+	(wire
+		(pts
 			(xy 121.92 45.72) (xy 121.92 93.98)
 		)
@@
 	(wire
 		(pts
+			(xy 285.75 76.2) (xy 285.75 95.25)
+		)
+		(stroke
+			(width 1)
+			(type default)
+			(color 73 152 255 1)
+		)
+	)
+	(wire
+		(pts
 			(xy 127 119.38) (xy 262.89 119.38)
 		)
@@
 		)
 		(stroke
-			(width 0)
-			(type default)
+			(width 1)
+			(type default)
+			(color 73 152 255 1)
 		)
 	)
@@
 		)
 		(stroke
-			(width 0)
-			(type default)
+			(width 1)
+			(type default)
+			(color 73 152 255 1)
 		)
 	)
@@
 	(wire
 		(pts
-			(xy 309.88 95.25) (xy 309.88 31.75)
-		)
-		(stroke
-			(width 0)
-			(type default)
-		)
-	)
-	(wire
-		(pts
 			(xy 307.34 95.25) (xy 307.34 34.29)
 		)
@@
 		)
 		(stroke
-			(width 0)
-			(type default)
-		)
-	)
-	(wire
-		(pts
-			(xy 309.88 31.75) (xy 111.76 31.75)
-		)
-		(stroke
-			(width 0)
-			(type default)
+			(width 1)
+			(type default)
+			(color 73 152 255 1)
 		)
 	)
@@
 			)
 			(justify left bottom)
+		)
+	)
+	(text "Do i need 2 pins for the HOST_RUN_PG? should it be a single one?"
+		(exclude_from_sim no)
+		(at 154.686 149.606 0)
+		(effects
+			(font
+				(size 1.27 1.27)
+			)
+			(justify left)
 		)
 	)
@@
 			)
 		)
-		(pin "+3.3v_HOST_PCIe" input
-			(at 309.88 95.25 90)
-			(effects
-				(font
-					(size 1.27 1.27)
-				)
-				(justify right)
-			)
-		)
 		(pin "+5v_HOST_HDMI" input
 			(at 307.34 95.25 90)
@@
 				)
 				(justify left)
+			)
+		)
+		(pin "+3v3_AUX" input
+			(at 285.75 95.25 90)
+			(effects
+				(font
+					(size 1.27 1.27)
+				)
+				(justify right)
 			)
 		)
@@
 			)
 		)
-		(pin "+3.3v_BMC" output
-			(at 102.87 93.98 90)
-			(effects
-				(font
-					(size 1.27 1.27)
-				)
-				(justify right)
-			)
-		)
 		(pin "BMC_HOST_BT_nDis" input
 			(at 127 133.35 0)
@@
 		(pin "BMC_UART1_RX" input
 			(at 127 166.37 0)
+			(effects
+				(font
+					(size 1.27 1.27)
+				)
+				(justify right)
+			)
+		)
+		(pin "+3v3_AUX" output
+			(at 102.87 93.98 90)
 			(effects
 				(font
@@
 			)
 		)
-		(pin "+3.3v_BMC" input
-			(at 102.87 63.5 270)
-			(effects
-				(font
-					(size 1.27 1.27)
-				)
-				(justify left)
-			)
-		)
 		(pin "BMC_I2C_0_SCK" input
 			(at 91.44 63.5 270)
@@
 			)
 		)
-		(pin "+3.3v_HOST_PCIe" output
-			(at 111.76 31.75 0)
-			(effects
-				(font
-					(size 1.27 1.27)
-				)
-				(justify right)
+		(pin "+3v3_AUX" input
+			(at 102.87 63.5 270)
+			(effects
+				(font
+					(size 1.27 1.27)
+				)
+				(justify left)
 			)
 		)
@@
 			)
 		)
-		(pin "+3.3v_BMC" output
+		(pin "+3v3_AUX" output
 			(at 48.26 95.25 90)
 			(effects
