File: kicad/mk2/srvant-mk2/bmc.kicad_sch (KiCad schematic)
At the start: 42 parts, among them J3 Conn_01x03, J4 USB_OTG, J7 Conn_02x05_Odd_Even, SW1 POWER, SW2 EMMC_KEY, SW3 RST, SW4 HOST_RESET, U22 TMP1075DSG, U25 74AHC1G08, U5 rp-t113-s3, U6 PCF85063AT/AAZ, U7 TPD4EUSB30, U8 74LVC2G07, Y1 X32K768S301

Commit message: redesign for the next version
Parts:
- removed R16: 47K, Resistor_SMD:R_0402_1005Metric, symbol Device:R
- removed R62, R63, R64, R69: 0, Resistor_SMD:R_0402_1005Metric, symbol Device:R
- removed SW2: EMMC_KEY, button-1571563-4:SW4_FSM-5P23_TEC, symbol Switch:SW_Push
- removed SW3: RST, button-1571563-4:SW4_FSM-5P23_TEC, symbol Switch:SW_Push
- removed U8: 74LVC2G07, Package_TO_SOT_SMD:SOT-23-6, symbol 74xGxx:74LVC2G07
- added D11: POWER, LED_SMD:LED_0603_1608Metric, symbol Device:LED
- added JP2, JP3, JP5, JP6: SolderJumper_2_Open, Jumper:SolderJumper-2_P1.3mm_Open_RoundedPad1.0x1.5mm, symbol Jumper:SolderJumper_2_Open
- added R77: 10K, Resistor_SMD:R_0402_1005Metric, symbol Device:R
- added SW2: FEL, SW4_FSM-5P23_TEC, symbol button-1571563-4:1571563-4
- added SW3: RST, SW4_FSM-5P23_TEC, symbol button-1571563-4:1571563-4
- C37: Field4 (none) -> Farnell; Field5 (none) -> 2611911; Field6 (none) -> RM EMK105 B7104KV-F; Field7 (none) -> TAIYO YUDEN EUROPE GMBH; Field8 (none) -> 110091611; digikey# EMK105B7104KV-F -> (none); farnell# 2611911 -> (none); manf# GRM155R71C104KA88 -> (none); mouser# 963-EMK105B7104KV-F -> (none)
- R11, R12, R71, R72: value 3.3K -> 10K
- R70: value 0 -> 1K; Field4 (none) -> Farnell; Field5 (none) -> 9239235; Field6 (none) -> RK73H1ETTP1001F; Field7 (none) -> KOA EUROPE GMBH; Field8 (none) -> 125049511; Part Description (none) -> Resistor 1K M1005 1% 63mW
- R73: value 0 -> 10K
Connections:
- net BMC_POWER_LED is gone; now on net BMC_ID_LED: U5.73 (PD16/LCD_D22/LVDS1_CKP/DMIC_DATA3/PWM0/PD_EINT16)
- net +5v_BMC: no longer U25.5 (VCC)
- net BMC_DEBUG_RX: now also U5.81 (PB7/LCD_D17/I2S2_MCLK/TWI3_SDA/IR_RX/LCD_D23/UART3_RX/CPUBIST1/PB_EINT7); no longer U5.63 (UART5_RX)
- net BMC_DEBUG_TX: now also U5.82 (PB6/LCD_D16/I2S2_LRCK/TWI3_SCK/PWM1/LCD_D22/UART3_TX/CPUBIST0/PB_EINT6); no longer U5.62 (UART5_TX)
- net BMC_HOST_BT_nDis: now also U5.57 (PD0/LCD_D2/LVDS0_V0P/DSI_D0P/TWI0_SCK/PD_EINT0); no longer U5.72 (PD_EINT15)
- net BMC_HOST_EEPROM_nWP: now also JP2.2 (B)
- net BMC_HOST_POST_COMPLETE: now also U5.58 (PD1/LCD_D3/LVDS0_V0N/DSI_D0N/UART2_TX/PD_EINT1); no longer U5.75 (PWM2)
- net BMC_HOST_POWER_BUTTON: now also U5.54 (PE1/NCSI0_VSYNC/UART2_CTS/TWI1_SDA/LCD_VSYNC/RGMII_RXD0/PE_EINT1); no longer U5.42 (PE_EINT13)
- net BMC_HOST_POWER_EN: now also JP5.2 (B)
- net BMC_HOST_POWER_OUT: now also U5.59 (PD2/LCD_D4/LVDS0_V1P/DSI_D1P/UART2_RX/PD_EINT2); no longer U5.76 (PWM3)
- net BMC_HOST_RESET_BUTTON: now also U5.55 (PE0/NCSI0_HSYNC/UART2_RTS/TWI1_SCK/LCD_HSYNC/RGMII_RXCTRL/PE_EINT0); no longer U5.43 (PE_EINT12)
- net BMC_HOST_RESET_OUT: now also U5.60 (PD3/LCD_D5/LVDS0_V1N/DSI_D1N/UART2_RTS/PD_EINT3)
- net BMC_HOST_USB_DEMUX_CONTROL: now also U5.85 (PB3/LCD_D1/I2S2_DOUT1/TWI0_SCK/I2S2_DIN0/LCD_D19/UART4_RX/CAN0_RX/PB_EINT3); no longer U5.50 (PE_EINT5)
- net BMC_HOST_WL_nDis: now also JP6.2 (B); no longer R70.1
- net BMC_HOST_nRPIBOOT: now also JP3.2 (B)
- net BMC_I2C_0_SCK: now also U5.53 (PE2/NCSI0_PCLK/UART2_TX/TWI0_SCK/CLK_FANOUT0/UART0_TX/RGMII_RXD1/PE_EINT2); no longer U5.85 (TWI0_SCK)
- net BMC_I2C_0_SDA: now also U5.52 (PE3/NCSI0_MCLK/UART2_RX/TWI0_SDA/CLK_FANOUT1/UART0_RX/RGMII_TXCK/PE_EINT3); no longer U5.86 (TWI0_SDA)
- net BMC_I2C_2_SCK: now also R11.2, U5.51 (PE4/NCSI0_D0/UART4_TX/TWI2_SCK/CLK_FANOUT2/D_JTAG_MS/RGMII_TXD0/PE_EINT4), U6.6 (SCL); no longer R71.1, U22.2 (SCL), U5.77 (TWI2_SCK)
- net BMC_I2C_2_SDA: now also R12.1, U5.50 (PE5/NCSI0_D1/UART4_RX/TWI2_SDA/LEDC_DO/D_JTAG_DI/RGMII_TXD1/PE_EINT5), U6.5 (SDA); no longer R72.1, U22.1 (SDA), U5.78 (TWI2_SDA)
- net BMC_I2C_3_SCK: now also R71.1, U22.2 (SCL), U5.49 (PE6/NCSI0_D2/UART5_TX/TWI3_SCK/OWA_IN/D_JTAG_DO/RGMII_TXCTRL/PE_EINT6); no longer R11.2, U5.82 (TWI3_SCK), U6.6 (SCL)
- net BMC_I2C_3_SDA: now also R72.1, U22.1 (SDA), U5.48 (PE7/NCSI0_D3/UART5_RX/TWI3_SDA/OWA_OUT/D_JTAG_CK/RGMII_CLKIN/PE_EINT7); no longer R12.1, U5.81 (TWI3_SDA), U6.5 (SDA)
- net BMC_ID_LED: now also R14.2; no longer U5.74 (PWM1)
- net BMC_TEMP_ALERT: now also U5.42 (PE13/TWI2_SDA/PWM5/DMIC_DATA3/RGMII_RXD2/PE_EINT13); no longer U5.79 (PWM7)
- net BMC_UART0_RX: now also U5.7 (PF4/SDC0_D3/UART0_RX/TWI0_SDA/PWM6/IR_TX/PF_EINT4); no longer U5.52 (UART0_RX)
- net BMC_UART0_TX: now also U5.5 (PF2/SDC0_CLK/UART0_TX/TWI0_SCK/LEDC_DO/OWA_IN/PF_EINT2); no longer U5.53 (UART0_TX)
- net BMC_USB_IDDET: now also U5.78 (PD21/LCD_VSYNC/TWI2_SDA/UART1_TX/PWM5/PD_EINT21); no longer J4.4 (ID), U5.71 (USB_DET)
- net EMMC_KEY: now also SW2.1, SW2.2
- net GND: now also D3.1 (K), D4.1 (K), D11.1 (K), SW3.1, SW3.2; no longer C37.2
- net NMI_N: now also C37.2; no longer R73.2
- net at U25.1: now also R73.2, SW3.3, SW3.4
- net at U25.2: now also C37.1, R77.2; no longer R73.1
- net 3.3v_BMC: now reaches R70.2
- net 3.3v_BMC: now also J7.3 (Pin_3), TP5.1, U5.30 (VCC-3V3); no longer U5.55 (PE_EINT0)
- net at U5.65 (PD8/LCD_D12/LVDS0_V3P/DSI_D3P/UART4_RX/PD_EINT8): now also JP5.1 (A)
- net at U5.66 (PD9/LCD_D13/LVDS0_V3N/DSI_D3N/PWM6/PD_EINT9): now also JP6.1 (A)
- net at R14.1: now also D4.2 (A); no longer D4.1 (K)
- net at R13.1: now also D3.2 (A); no longer D3.1 (K)
- net BMC_USER_LED: now reaches R13.2
- net BMC_USER_LED: now also U5.74 (PD17/LCD_D23/LVDS1_CKN/DMIC_DATA2/PWM1/PD_EINT17)
- net +3.3v_BMC renamed +3v3_AUX
- net +3v3_AUX: now also R73.1, U25.5 (VCC), R77.1, SW2.3, SW2.4; no longer C37.1, D3.2 (A), D4.2 (A), J7.3 (Pin_3), TP5.1, U5.30 (VCC-3V3)
- new net: JP3.1 (A), U5.61 (PD4/LCD_D6/LVDS0_V2P/DSI_CKP/UART2_CTS/PD_EINT4)
- new net: JP2.1 (A), U5.86 (PB2/LCD_D0/I2S2_DOUT2/TWI0_SDA/I2S2_DIN2/LCD_D18/UART4_TX/CAN0_TX/PB_EINT2)
- new net: D11.2 (A), R70.1
- new net CLK125_OUT: U5.120 (PG13/I2S1_BCLK/TWI0_SDA/RGMII_CLKIN/PWM2/LEDC_DO/UART1_RX/PG_EINT13)
- new net EPHY_25M: U5.129 (PG11/I2S1_MCLK/TWI3_SDA/EPHY_25M/CLK_FANOUT1/TCON_TRIG/PG_EINT11)
- new net MAC_RESET_OUT_N: U5.77 (PD20/LCD_HSYNC/TWI2_SCK/DMIC_CLK/PWM4/PD_EINT20)
- new net PHY_INT_N: U5.76 (PD19/LCD_DE/LVDS1_V3N/DMIC_DATA0/PWM3/PD_EINT19)
- new net PHY_MDC: U5.119 (PG14/I2S1_DIN0/TWI2_SCK/RGMII_MDC/I2S1_DOUT1/SPI0_WP/UART1_RTS/PG_EINT14)
- new net PHY_MDIO: U5.118 (PG15/I2S1_DOUT0/TWI2_SDA/RGMII_MDIO/I2S1_DIN1/SPI0_HOLD/UART1_CTS/PG_EINT15)
- new net RXC: U5.124 (PG10/PWM3/TWI3_SCK/RGMII_RXCK/CLK_FANOUT0/IR_RX/PG_EINT10)
- new net RXD0: U5.122 (PG1/SDC1_CMD/UART3_TX/RGMII_RXD0/PWM6/PG_EINT1)
- new net RXD1: U5.123 (PG2/SDC1_D0/UART3_RTS/RGMII_RXD1/UART4_TX/PG_EINT2)
- new net RXD2: U5.131 (PG8/UART1_RTS/TWI1_SCK/RGMII_RXD2/UART3_TX/PG_EINT8)
- new net RXD3: U5.130 (PG9/UART1_CTS/TWI1_SDA/RGMII_RXD3/UART3_RX/PG_EINT9)
- new net RX_CTL: U5.121 (PG0/SDC1_CLK/UART3_TX/RGMII_RXCTRL/PWM7/PG_EINT0)
- new net TXC: U5.125 (PG3/SDC1_D1/UART3_CTS/RGMII_TXCK/UART4_RX/PG_EINT3)
- new net TXD0: U5.126 (PG4/SDC1_D2/UART5_TX/RGMII_TXD0/PWM5/PG_EINT4)
- new net TXD1: U5.127 (PG5/SDC1_D3/UART5_RX/RGMII_TXD1/PWM4/PG_EINT5)
- new net TXD2: U5.133 (PG6/UART1_TX/TWI2_SCK/RGMII_TXD2/PWM1/PG_EINT6)
- new net TXD3: U5.132 (PG7/UART1_RX/TWI2_SDA/RGMII_TXD3/OWA_IN/PG_EINT7)
- new net TX_CTL: U5.128 (PG12/I2S1_LRCK/TWI0_SCK/RGMII_TXCTRL/CLK_FANOUT2/PWM0/UART1_TX/PG_EINT12)
Other:
- note added: "BMC_POWER_LED"
- moved on the sheet: D3, D4, D9, FB1, J4, R13, R14, SW1, SW4, U25, U7

Commit message: state
Parts:
- added JP4: SolderJumper_2_Open, Jumper:SolderJumper-2_P1.3mm_Open_RoundedPad1.0x1.5mm, symbol Jumper:SolderJumper_2_Open
Connections:
- net BMC_HOST_USB_DEMUX_CONTROL: now also JP4.2 (B); no longer U5.85 (PB3/LCD_D1/I2S2_DOUT1/TWI0_SCK/I2S2_DIN0/LCD_D19/UART4_RX/CAN0_RX/PB_EINT3)
- new net: JP4.1 (A), U5.85 (PB3/LCD_D1/I2S2_DOUT1/TWI0_SCK/I2S2_DIN0/LCD_D19/UART4_RX/CAN0_RX/PB_EINT3)
Changed lines of the file:
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@@
 	(wire
 		(pts
+			(xy 185.42 93.98) (xy 195.58 93.98)
+		)
+		(stroke
+			(width 0)
+			(type default)
+		)
+	)
+	(wire
+		(pts
 			(xy 182.88 85.09) (xy 195.58 85.09)
 		)
@@
 	(wire
 		(pts
-			(xy 172.72 93.98) (xy 195.58 93.98)
+			(xy 172.72 93.98) (xy 177.8 93.98)
 		)
 		(stroke
@@
 					(unit 1)
 				)
+			)
+		)
+	)
+	(symbol
+		(lib_id "Jumper:SolderJumper_2_Open")
+		(at 181.61 93.98 0)
+		(mirror y)
+		(unit 1)
+		(exclude_from_sim yes)
+		(in_bom no)
+		(on_board yes)
+		(dnp no)
+		(property "Reference" "JP4"
+			(at 184.404 92.71 0)
+			(effects
+				(font
+					(size 1.27 1.27)
+				)
+			)
+		)
+		(property "Value" "SolderJumper_2_Open"
+			(at 182.88 94.996 0)
+			(effects
+				(font
+					(size 1.27 1.27)
+				)
+				(hide yes)
+			)
+		)
+		(property "Footprint" "Jumper:SolderJumper-2_P1.3mm_Open_RoundedPad1.0x1.5mm"
+			(at 181.61 93.98 0)
+			(effects
+				(font
+					(size 1.27 1.27)
+				)
+				(hide yes)
+			)
+		)
+		(property "Datasheet" "~"
+			(at 181.61 93.98 0)
+			(effects
+				(font
+					(size 1.27 1.27)
+				)
+				(hide yes)
+			)
+		)
+		(property "Description" "Solder Jumper, 2-pole, open"
+			(at 181.61 93.98 0)
+			(effects
+				(font
+					(size 1.27 1.27)
+				)
+				(hide yes)
+			)
+		)
+		(pin "1"
+		)
+		(pin "2"
+		)
+		(instances
+			(project "srvant-mk2"
+				(path "/1859a578-b791-4142-bdf4-fda494df1146/a3ddce6d-c94c-48a5-9fee-a70fbee730bf"
+					(reference "JP4")
+					(unit 1)
+				)
