File: kicad/cm4/srvant-mk2.kicad_sch (KiCad schematic)
At the start: 123 parts, among them J1 Screw_Terminal_01x02, J10 HDMI connector, J14 JST_SHBM04B-SRSS-TB, J2 USB_B_Micro, J3 USB3_A, J4 Screw_Terminal_01x02, J5 Conn_01x03, J6 Conn_01x03, J7 ARJM11, J8 Bus_M.2_Socket_M, J9 Conn_02x10_Odd_Even, Q1 CSD17307Q5A, Q2 CSD18502Q5B, U1 INA219AxDCN, U10 ASEK-32.768KHZ-L-R-T, U2 AP63205WU, U3 LM3150MH, U4 TPD4EUSB30, U5 TPD4EUSB30, U6 SLB9670VQ20FW785XTMA1, U7 AP22653W6, U8 74LVC1G07SE-7, U9 RT9742SNGV

Commit message: state of the cm4(5), manufactured revision
Parts:
- removed RTCK1: RTCK, TestPoint:TestPoint_Pad_D1.0mm, symbol Connector:TestPoint
- removed TCK1: TCK, TestPoint:TestPoint_Pad_D1.0mm, symbol Connector:TestPoint
- removed TDI1: TDI, TestPoint:TestPoint_Pad_D1.0mm, symbol Connector:TestPoint
- removed TDO1: TDO, TestPoint:TestPoint_Pad_D1.0mm, symbol Connector:TestPoint
- removed TMS1: TMS, TestPoint:TestPoint_Pad_D1.0mm, symbol Connector:TestPoint
- removed TP6, TP7: PCIe_nRST, TestPoint:TestPoint_Pad_D1.0mm, symbol Connector:TestPoint
- removed TRST1: TRST, TestPoint:TestPoint_Pad_D1.0mm, symbol Connector:TestPoint
- added TP11: PCIe_nCLKREQ, TestPoint:TestPoint_Pad_D1.0mm, symbol Connector:TestPoint
- J7: footprint Connector_RJ:RJ45_Wuerth_7499111446_Horizontal -> Connector_RJ:RJ45_Pulse_JK0654219NL_Horizontal
- U7: Field5 31-AP22653W6-7CT-ND -> AP2553W6-7DICT-ND
Connections:
- net PCIE_nCLKREQ is gone; now on net PCIE_CLK_nREQ: Module1.102 (PCIe_nCLKREQ)
- net PCIE_nWAKE is gone; now on net PCIE_WAKE: Module1.104 (PCIE_nWAKE)
- net SENSE_IN- is gone; now on net +5v_HOST: R1.1, R3.1
- net +3.3v_HOST: now also C4.1, C5.1, R6.1, R8.1, U1.4 (VS)
- net +3v3 (BMC): no longer C4.1, C5.1, R6.1, R8.1, U1.4 (VS)
- net +5v_HOST: no longer C1.1, C2.1, J2.1 (VBUS), R1.2, R2.1
- net HDMI0_HOTPLUG: now also Module1.153 (HDMI0_HOTPLUG)
- net PCIE_WAKE: now also TP11.1
- net at J5.1 (Pin_1): now also R7.2; no longer R5.1
- net at J5.3 (Pin_3): now also R5.1; no longer R7.2
- net CAM_GPIO1: no longer names the net of Module1.100 (CAM_GPIO1)
- net CC1: no longer names the net of Module1.94 (CC1)
- net CC2: no longer names the net of Module1.96 (CC2)
- net HOST_UART_RX renamed BMC_HOST_UART_TX
- net HOST_UART_TX renamed BMC_HOST_UART_RX
- net SCL0 renamed BMC_HOST_I2C_SCK
- net SDA0 renamed BMC_HOST_I2C_SDA
- new net +5v_IN: C1.1, C2.1, J2.1 (VBUS), R1.2, R2.1
- no-connect marks 56 -> 57
Other:
- note removed: "HOST JTAG"
- moved on the sheet: D2, TP3
